Commit message: chore: tunning

File: rm_simulation/pb_rm_simulation/urdf/simulation_waking_robot.xacro (robot description, xacro)
@@ -108,5 +108,4 @@
         <axis xyz="0 0 1" />
         <anchor xyz="0 0 0" />
-        <limit effort="100" velocity="100" />
         <parent link="base_link"/>
         <child link="wheel_2"/>
@@ -179,14 +178,8 @@
                 <remapping>odom:=state_estimation</remapping>
             </ros>
-            <update_rate>100</update_rate>
-            <publish_rate>100</publish_rate>
+            <update_rate>20</update_rate>
+            <publish_rate>20</publish_rate>
             <publish_odom>false</publish_odom>
             <publish_odom_tf>false</publish_odom_tf>
-            <leftFrontJoint>base_to_wheel1</leftFrontJoint>
-            <rightFrontJoint>base_to_wheel3</rightFrontJoint>
-            <leftRearJoint>base_to_wheel2</leftRearJoint>
-            <rightRearJoint>base_to_wheel4</rightRearJoint>
-            <wheelSeparation>0.26</wheelSeparation>
-            <wheelDiameter>0.12</wheelDiameter>
             <odometry_frame>odom</odometry_frame>
             <robot_base_frame>base_link</robot_base_frame>

Commit message: fix: wrongly deleted some packages

File: rm_simulation/pb_rm_simulation/urdf/simulation_waking_robot.xacro (robot description, xacro)
@@ -29,4 +29,11 @@
         <xacro:default_inertial mass="8.2"/>
     </link>
+    <link name="yaw_link"/>
+    <joint name="base_to_yaw" type="continuous">
+        <parent link="base_link"/>
+        <child link="yaw_link"/>
+        <origin rpy="0 0 0" xyz="0 0 0.1"/>
+        <axis xyz="0 0 1" />
+    </joint>
     <link name="wheel_1">
         <visual>

Commit message: 3d导航，无法到达目标点，卡死在接受结果反馈阶段

File: rm_simulation/pb_rm_simulation/urdf/simulation_waking_robot.xacro (robot description, xacro)
@@ -179,5 +179,6 @@
     <!-- Drive controller -->
     <gazebo>
-        <plugin name="mecanum_controller" filename="libgazebo_ros_planar_move.so">
+        <plugin name="mecanum_controller" filename="/home/sentry_ws/src/rm_simulation/pb_rm_simulation/RC_vision_2026/gazebo_for_humble/install/my_gazebo_plugins/lib/libcmd_vel_z_plugin.so">
+        <!-- <plugin name="mecanum_controller" filename="libgazebo_ros_planar_move.so"> -->
             <ros>
                 <!-- <namespace>/demo</namespace> -->
@@ -196,8 +197,13 @@
     <gazebo reference="imu_link">
         <material>Gazebo/Orange</material>
-        <gravity>true</gravity>
+        <gravity>false</gravity>
         <sensor name="imu_sensor" type="imu">
             <always_on>true</always_on>
             <update_rate>200</update_rate>
+            <!-- 关键：开启重力补偿，即使Gazebo无重力，也让IMU输出模拟重力的z轴加速度 -->
+            <!-- <gravity_compensation>true</gravity_compensation> -->
+            <!-- 手动设置模拟重力的加速度（z轴向下为负，对应-9.8m/s²） -->
+            <!-- <xacro:property name="sim_gravity_z" value="-9.8" /> -->
+            <!-- <linear_acceleration_bias>0 0 ${sim_gravity_z}</linear_acceleration_bias> -->
             <visualize>true</visualize>
             <topic>__default_topic__</topic>
